File: hardware/connection.kicad_sch (KiCad schematic)
At the start: 20 parts, among them J3 Conn_Buttons, J6 Conn_Controller

Commit message: ✨ Final PCB updates
Parts:
- renumbered C14 to C301, C15 to C302, C16 to C303, D1 to D301, D3 to D302, D2 to D303, F2 to F301, J6 to J2, R26 to R301, R27 to R302, R28 to R303, R29 to R304, R55 to R305, R54 to R306, R53 to R307, R52 to R308, TP7 to TP301, TP9 to TP302, TP8 to TP303
Changed lines of the file:
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@@
 		(on_board yes)
 		(dnp no)
-		(property "Reference" "TP9"
+		(property "Reference" "TP302"
 			(at 69.342 52.578 0)
 			(effects
@@
 			(project "peak"
 				(path "/54a54a18-4a65-4728-b17a-32b4a97370c1/7b8eb5a1-fed9-4601-b83f-2313cfb612ed"
-					(reference "TP9")
+					(reference "TP302")
 					(unit 1)
 				)
@@
 		(on_board yes)
 		(dnp no)
-		(property "Reference" "TP8"
+		(property "Reference" "TP303"
 			(at 61.468 29.972 0)
 			(effects
@@
 			(project "peak"
 				(path "/54a54a18-4a65-4728-b17a-32b4a97370c1/7b8eb5a1-fed9-4601-b83f-2313cfb612ed"
-					(reference "TP8")
+					(reference "TP303")
 					(unit 1)
 				)
@@
 		(dnp no)
 		(fields_autoplaced yes)
-		(property "Reference" "#PWR0116"
+		(property "Reference" "#PWR0121"
 			(at 143.51 48.26 0)
 			(effects
@@
 			(project "peak"
 				(path "/54a54a18-4a65-4728-b17a-32b4a97370c1/7b8eb5a1-fed9-4601-b83f-2313cfb612ed"
-					(reference "#PWR0116")
+					(reference "#PWR0121")
 					(unit 1)
 				)
@@
 		(dnp no)
 		(fields_autoplaced yes)
-		(property "Reference" "J6"
+		(property "Reference" "J2"
 			(at 97.79 30.48 90)
 			(effects
@@
 			(project ""
 				(path "/54a54a18-4a65-4728-b17a-32b4a97370c1/7b8eb5a1-fed9-4601-b83f-2313cfb612ed"
-					(reference "J6")
+					(reference "J2")
 					(unit 1)
 				)
@@
 		(on_board yes)
 		(dnp no)
-		(property "Reference" "R26"
+		(property "Reference" "R301"
 			(at 39.37 58.42 90)
 			(effects
@@
 			(project ""
 				(path "/54a54a18-4a65-4728-b17a-32b4a97370c1/7b8eb5a1-fed9-4601-b83f-2313cfb612ed"
-					(reference "R26")
+					(reference "R301")
 					(unit 1)
 				)
@@
 		(on_board yes)
 		(dnp no)
-		(property "Reference" "C14"
+		(property "Reference" "C301"
 			(at 57.404 38.354 0)
 			(effects
@@
 			(project ""
 				(path "/54a54a18-4a65-4728-b17a-32b4a97370c1/7b8eb5a1-fed9-4601-b83f-2313cfb612ed"
-					(reference "C14")
+					(reference "C301")
 					(unit 1)
 				)
@@
 		(dnp no)
 		(fields_autoplaced yes)
-		(property "Reference" "D3"
+		(property "Reference" "D302"
 			(at 153.67 26.67 90)
 			(effects
@@
 			(project ""
 				(path "/54a54a18-4a65-4728-b17a-32b4a97370c1/7b8eb5a1-fed9-4601-b83f-2313cfb612ed"
-					(reference "D3")
+					(reference "D302")
 					(unit 1)
 				)
@@
 		(dnp no)
 		(fields_autoplaced yes)
-		(property "Reference" "#PWR0104"
+		(property "Reference" "#PWR0122"
 			(at 119.38 50.8 0)
 			(effects
@@
 			(project ""
 				(path "/54a54a18-4a65-4728-b17a-32b4a97370c1/7b8eb5a1-fed9-4601-b83f-2313cfb612ed"
-					(reference "#PWR0104")
+					(reference "#PWR0122")
 					(unit 1)
 				)
@@
 		(on_board yes)
 		(dnp no)
-		(property "Reference" "TP7"
+		(property "Reference" "TP301"
 			(at 28.448 29.972 0)
 			(effects
@@
 			(project "peak"
 				(path "/54a54a18-4a65-4728-b17a-32b4a97370c1/7b8eb5a1-fed9-4601-b83f-2313cfb612ed"
-					(reference "TP7")
+					(reference "TP301")
 					(unit 1)
 				)
@@
 		(on_board yes)
 		(dnp no)
-		(property "Reference" "D1"
+		(property "Reference" "D301"
 			(at 41.656 39.37 90)
 			(effects
@@
 			(project ""
 				(path "/54a54a18-4a65-4728-b17a-32b4a97370c1/7b8eb5a1-fed9-4601-b83f-2313cfb612ed"
-					(reference "D1")
+					(reference "D301")
 					(unit 1)
 				)
@@
 		(dnp no)
 		(fields_autoplaced yes)
-		(property "Reference" "#PWR0117"
+		(property "Reference" "#PWR0126"
 			(at 171.45 40.64 0)
 			(effects
@@
 			(project ""
 				(path "/54a54a18-4a65-4728-b17a-32b4a97370c1/7b8eb5a1-fed9-4601-b83f-2313cfb612ed"
-					(reference "#PWR0117")
+					(reference "#PWR0126")
 					(unit 1)
 				)
@@
 		(dnp no)
 		(fields_autoplaced yes)
-		(property "Reference" "#PWR0115"
+		(property "Reference" "#PWR0127"
 			(at 177.8 88.9 0)
 			(effects
@@
 			(project "peak"
 				(path "/54a54a18-4a65-4728-b17a-32b4a97370c1/7b8eb5a1-fed9-4601-b83f-2313cfb612ed"
-					(reference "#PWR0115")
+					(reference "#PWR0127")
 					(unit 1)
 				)
@@
 		(on_board yes)
 		(dnp no)
-		(property "Reference" "#PWR029"
+		(property "Reference" "#PWR0123"
 			(at 92.71 40.64 0)
 			(effects
@@
 			(project ""
 				(path "/54a54a18-4a65-4728-b17a-32b4a97370c1/7b8eb5a1-fed9-4601-b83f-2313cfb612ed"
-					(reference "#PWR029")
+					(reference "#PWR0123")
 					(unit 1)
 				)
@@
 		(on_board yes)
 		(dnp no)
-		(property "Reference" "R55"
+		(property "Reference" "R305"
 			(at 161.29 54.61 90)
 			(effects
@@
 			(project "peak"
 				(path "/54a54a18-4a65-4728-b17a-32b4a97370c1/7b8eb5a1-fed9-4601-b83f-2313cfb612ed"
-					(reference "R55")
+					(reference "R305")
 					(unit 1)
 				)
@@
 		(on_board yes)
 		(dnp yes)
-		(property "Reference" "R28"
+		(property "Reference" "R303"
 			(at 40.64 76.2 90)
 			(effects
@@
 			(project "peak"
 				(path "/54a54a18-4a65-4728-b17a-32b4a97370c1/7b8eb5a1-fed9-4601-b83f-2313cfb612ed"
-					(reference "R28")
+					(reference "R303")
 					(unit 1)
 				)
@@
 		(on_board yes)
 		(dnp no)
-		(property "Reference" "C15"
+		(property "Reference" "C302"
 			(at 32.258 101.854 0)
 			(effects
@@
 			(project "peak"
 				(path "/54a54a18-4a65-4728-b17a-32b4a97370c1/7b8eb5a1-fed9-4601-b83f-2313cfb612ed"
-					(reference "C15")
+					(reference "C302")
 					(unit 1)
 				)
@@
 		(on_board yes)
 		(dnp no)
-		(property "Reference" "R27"
+		(property "Reference" "R302"
 			(at 39.37 60.96 90)
 			(effects
@@
 			(project "peak"
 				(path "/54a54a18-4a65-4728-b17a-32b4a97370c1/7b8eb5a1-fed9-4601-b83f-2313cfb612ed"
-					(reference "R27")
+					(reference "R302")
 					(unit 1)
 				)
@@
 		(on_board yes)
 		(dnp no)
-		(property "Reference" "R54"
+		(property "Reference" "R306"
 			(at 161.29 58.42 90)
 			(effects
@@
 			(project "peak"
 				(path "/54a54a18-4a65-4728-b17a-32b4a97370c1/7b8eb5a1-fed9-4601-b83f-2313cfb612ed"
-					(reference "R54")
+					(reference "R306")
 					(unit 1)
 				)
@@
 		(dnp no)
 		(fields_autoplaced yes)
-		(property "Reference" "#PWR039"
+		(property "Reference" "#PWR0118"
 			(at 69.85 39.37 0)
 			(effects
@@
 			(project "peak"
 				(path "/54a54a18-4a65-4728-b17a-32b4a97370c1/7b8eb5a1-fed9-4601-b83f-2313cfb612ed"
-					(reference "#PWR039")
+					(reference "#PWR0118")
 					(unit 1)
 				)
@@
 		(on_board yes)
 		(dnp no)
-		(property "Reference" "D2"
+		(property "Reference" "D303"
 			(at 168.2115 71.12 0)
 			(effects
@@
 			(project ""
 				(path "/54a54a18-4a65-4728-b17a-32b4a97370c1/7b8eb5a1-fed9-4601-b83f-2313cfb612ed"
-					(reference "D2")
+					(reference "D303")
 					(unit 1)
 				)
@@
 		(on_board yes)
 		(dnp no)
-		(property "Reference" "R52"
+		(property "Reference" "R308"
 			(at 167.64 40.64 90)
 			(effects
@@
 			(project "peak"
 				(path "/54a54a18-4a65-4728-b17a-32b4a97370c1/7b8eb5a1-fed9-4601-b83f-2313cfb612ed"
-					(reference "R52")
+					(reference "R308")
 					(unit 1)
 				)
@@
 		(on_board yes)
 		(dnp no)
-		(property "Reference" "#PWR043"
+		(property "Reference" "#PWR0120"
 			(at 35.56 35.56 0)
 			(effects
@@
 			(project "peak"
 				(path "/54a54a18-4a65-4728-b17a-32b4a97370c1/7b8eb5a1-fed9-4601-b83f-2313cfb612ed"
-					(reference "#PWR043")
+					(reference "#PWR0120")
 					(unit 1)
 				)
@@
 		(on_board yes)
 		(dnp no)
-		(property "Reference" "R53"
+		(property "Reference" "R307"
 			(at 161.29 62.23 90)
 			(effects
@@
 			(project "peak"
 				(path "/54a54a18-4a65-4728-b17a-32b4a97370c1/7b8eb5a1-fed9-4601-b83f-2313cfb612ed"
-					(reference "R53")
+					(reference "R307")
 					(unit 1)
 				)
@@
 		(dnp no)
 		(fields_autoplaced yes)
-		(property "Reference" "#PWR037"
+		(property "Reference" "#PWR0119"
 			(at 69.85 53.34 0)
 			(effects
@@
 			(project "peak"
 				(path "/54a54a18-4a65-4728-b17a-32b4a97370c1/7b8eb5a1-fed9-4601-b83f-2313cfb612ed"
-					(reference "#PWR037")
+					(reference "#PWR0119")
 					(unit 1)
 				)
@@
 		(on_board yes)
 		(dnp no)
-		(property "Reference" "C16"
+		(property "Reference" "C303"
 			(at 39.878 101.854 0)
 			(effects
@@
 			(project "peak"
 				(path "/54a54a18-4a65-4728-b17a-32b4a97370c1/7b8eb5a1-fed9-4601-b83f-2313cfb612ed"
-					(reference "C16")
+					(reference "C303")
 					(unit 1)
 				)
@@
 		(on_board yes)
 		(dnp yes)
-		(property "Reference" "R29"
+		(property "Reference" "R304"
 			(at 40.64 78.74 90)
 			(effects
@@
 			(project "peak"
 				(path "/54a54a18-4a65-4728-b17a-32b4a97370c1/7b8eb5a1-fed9-4601-b83f-2313cfb612ed"
-					(reference "R29")
+					(reference "R304")
 					(unit 1)
 				)
@@
 		(dnp no)
 		(fields_autoplaced yes)
-		(property "Reference" "#PWR041"
+		(property "Reference" "#PWR0125"
 			(at 35.56 100.33 0)
 			(effects
@@
 			(project "peak"
 				(path "/54a54a18-4a65-4728-b17a-32b4a97370c1/7b8eb5a1-fed9-4601-b83f-2313cfb612ed"
-					(reference "#PWR041")
+					(reference "#PWR0125")
 					(unit 1)
 				)
@@
 		(dnp no)
 		(fields_autoplaced yes)
-		(property "Reference" "#PWR042"
+		(property "Reference" "#PWR0124"
 			(at 35.56 116.84 0)
 			(effects
@@
 			(project "peak"
 				(path "/54a54a18-4a65-4728-b17a-32b4a97370c1/7b8eb5a1-fed9-4601-b83f-2313cfb612ed"
-					(reference "#PWR042")
+					(reference "#PWR0124")
 					(unit 1)
 				)
@@
 		(on_board yes)
 		(dnp no)
-		(property "Reference" "F2"
+		(property "Reference" "F301"
 			(at 38.1 33.528 90)
 			(effects
@@
 			(project ""
 				(path "/54a54a18-4a65-4728-b17a-32b4a97370c1/7b8eb5a1-fed9-4601-b83f-2313cfb612ed"
-					(reference "F2")
-					(unit 1)
-				)
+					(reference "F301")
+					(unit 1)
+				)
