File: hardware/peak.kicad_pcb (KiCad board)
At the start: 6 copper layers, 47 x 69.4 mm, 153 parts, among them J2 Conn_DEBUG_C6, J3 Conn_Buttons, J4 Conn_DEBUG_P4, J6 Conn_Controller, Q1 DMP10H400SE, Q2 BSS123, U11 LTR-329ALS-01, U12 ESP32-C6-MINI-1/U, U2 AP63203WU, U3 MCP2542FDxMF, U4 TPS62A04ADRL, U5 PLMR51635XDDCR, U6 AP3019AKTR, U7 W25Q128JVP, U8 T117, U9 74LVC1G17, X1 ECS-400-10-37B2-CKY-TR

Commit message: ✨ Finish rev 1.1
Parts:
- removed the TP9 at (208.8, 128.5)
- added TP6: 3.3VA, TestPoint:TestPoint_Pad_D1.0mm, F.Cu at (198.2, 81.9)
- added TP9: GND, TestPoint:TestPoint_Pad_D1.0mm, F.Cu at (210.1, 128.9)
- added TP9: GND, TestPoint:TestPoint_Pad_D1.0mm, F.Cu at (198.5, 68.2)
- added TP9: GND, TestPoint:TestPoint_Pad_D1.0mm, F.Cu at (217.9, 99.2)
- added TP9: GND, TestPoint:TestPoint_Pad_D1.0mm, F.Cu at (218.4, 68.4)
- moved TP2 20.2 mm to (218.3, 81.9)
- moved TP7 14.5 mm to (196.8, 112.2)
- moved C40 6.49 mm to (206.9, 82.6)
- moved C39 4.87 mm to (205.0, 82.6)
- moved C57 4.77 mm to (201.2, 85.5), turned to 180 degrees
- moved C58 4.75 mm to (201.2, 84.5), turned to 180 degrees
- moved C32 3.17 mm to (198.0, 79.2), turned to -90 degrees
- moved X1 2.82 mm to (202.8, 81.5)
- moved C33 2.57 mm to (199.6, 79.2), turned to -90 degrees
- moved FB1 2.56 mm to (199.0, 76.8), turned to 0 degrees
- moved TP3 2.33 mm to (228.2, 84.9)
- moved TP4 2.21 mm to (228.7, 97.9)
- moved TP1 2.10 mm to (188.6, 85.1)
- moved C61 1.70 mm to (199.0, 70.7)
- moved R22 0.77 mm to (206.5, 81.1)
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Connections:
- C39 pad 1: Net-(C39-Pad1) -> /MCU/XTAL_P
- C40 pad 1: Net-(C40-Pad1) -> /MCU/XTAL_N
- R21 pad 2: Net-(C39-Pad1) -> Net-(R21-Pad2)
- R22 pad 1: Net-(C40-Pad1) -> Net-(R22-Pad1)
- X1 pad 1: Net-(C39-Pad1) -> Net-(R21-Pad2)
- X1 pad 3: Net-(C40-Pad1) -> Net-(R22-Pad1)
Routing:
- net +5V: track 0.00 -> 128.8 mm, vias 0 -> 10
- net +3.3V: track 0.00 -> 121.0 mm, vias 0 -> 26
- net /IO/SDA_MCU: track 0.00 -> 77.9 mm, vias 0 -> 4
- net /IO/SCL_MCU: track 0.00 -> 77.6 mm, vias 0 -> 4
- net Net-(C13-Pad1): track 0.00 -> 64.3 mm, vias 0 -> 3
- net /Connection/Button_D: track 0.00 -> 57.1 mm, vias 0 -> 3
- net /Connection/Button_P: track 0.00 -> 54.5 mm, vias 0 -> 3
- net /Connection/Button_U: track 0.00 -> 50.2 mm, vias 0 -> 3
- net +1V2: track 0.00 -> 43.3 mm, vias 0 -> 4
- net /Connection/TX/CANL: track 0.00 -> 38.6 mm, vias 0 -> 3
- net /MCU/EN: track 0.00 -> 37.0 mm, vias 0 -> 2
- net /Display/LEDA: track 0.00 -> 34.5 mm, vias 0 -> 2
- net /Connection/RX/CANH: track 0.00 -> 34.2 mm, vias 0 -> 3
- net /Display/LED_PWM: track 0.00 -> 33.3 mm, vias 0 -> 2
- net /IO/SW_MCU: track 0.00 -> 33.2 mm, vias 0 -> 2
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- added copper zone on In2.Cu, net VBUS
Other:
- board text added: "3.3VA"
- board text added: "BAT+"
- board text added: "D"
- board text added: "G"
- board text added: "GND"
- board text added: "LEDA"
- board text added: "P"
- board text added: "R"
- board text added: "S"
- board text added: "T"
- board text added: "U"
- board text added: "V"
- board text added: "VBUS"

Commit message: 🔨 Update the pcb
Parts:
- moved TP3 30.4 mm to (198.5, 91.4)
Routing:
- net +1V2: track 43.3 -> 48.5 mm
Changed lines of the file:
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@@
 		)
 	)
+	(footprint "TestPoint:TestPoint_Pad_D1.0mm"
+		(layer "F.Cu")
+		(at 198.5031 91.400001)
+		(descr "SMD pad as test Point, diameter 1.0mm")
+		(tags "test point SMD pad")
+		(property "Reference" "TP3"
+			(at 0 -1.448 0)
+			(layer "F.SilkS")
+			(hide yes)
+			(effects
+				(font
+					(size 1 1)
+					(thickness 0.15)
+				)
+			)
+		)
+		(property "Value" "1.2V"
+			(at 0 1.55 0)
+			(layer "F.Fab")
+			(hide yes)
+			(effects
+				(font
+					(size 1 1)
+					(thickness 0.15)
+				)
+			)
+		)
+		(property "Datasheet" "~"
+			(at 0 0 0)
+			(unlocked yes)
+			(layer "F.Fab")
+			(hide yes)
+			(effects
+				(font
+					(size 1.27 1.27)
+					(thickness 0.15)
+				)
+			)
+		)
+		(property "Description" "test point"
+			(at 0 0 0)
+			(unlocked yes)
+			(layer "F.Fab")
+			(hide yes)
+			(effects
+				(font
+					(size 1.27 1.27)
+					(thickness 0.15)
+				)
+			)
+		)
+		(attr exclude_from_pos_files)
+		(fp_circle
+			(center 0 0)
+			(end 0 0.7)
+			(stroke
+				(width 0.12)
+				(type solid)
+			)
+			(fill no)
+			(layer "F.SilkS")
+		)
+		(fp_circle
+			(center 0 0)
+			(end 1 0)
+			(stroke
+				(width 0.05)
+				(type solid)
+			)
+			(fill no)
+			(layer "F.CrtYd")
+		)
+		(pad "1" smd circle
+			(at 0 0)
+			(size 1 1)
+			(layers "F.Cu" "F.Mask")
+			(net 6 "+1V2")
+			(pinfunction "1")
+			(pintype "passive")
+		)
+		(embedded_fonts no)
+	)
 	(footprint "Resistor_SMD:R_0603_1608Metric"
 		(layer "F.Cu")
@@
 		)
 	)
-	(footprint "TestPoint:TestPoint_Pad_D1.0mm"
-		(layer "F.Cu")
-		(at 228.2031 84.900001)
-		(descr "SMD pad as test Point, diameter 1.0mm")
-		(tags "test point SMD pad")
-		(property "Reference" "TP3"
-			(at 0 -1.448 0)
-			(layer "F.SilkS")
-			(hide yes)
-			(effects
-				(font
-					(size 1 1)
-					(thickness 0.15)
-				)
-			)
-		)
-		(property "Value" "1.2V"
-			(at 0 1.55 0)
-			(layer "F.Fab")
-			(hide yes)
-			(effects
-				(font
-					(size 1 1)
-					(thickness 0.15)
-				)
-			)
-		)
-		(property "Datasheet" "~"
-			(at 0 0 0)
-			(unlocked yes)
-			(layer "F.Fab")
-			(hide yes)
-			(effects
-				(font
-					(size 1.27 1.27)
-					(thickness 0.15)
-				)
-			)
-		)
-		(property "Description" "test point"
-			(at 0 0 0)
-			(unlocked yes)
-			(layer "F.Fab")
-			(hide yes)
-			(effects
-				(font
-					(size 1.27 1.27)
-					(thickness 0.15)
-				)
-			)
-		)
-		(property ki_fp_filters "Pin* Test*")
-		(sheetname "/Power supply/")
-		(sheetfile "power_supply.kicad_sch")
-		(attr exclude_from_pos_files)
-		(fp_circle
-			(center 0 0)
-			(end 0 0.7)
-			(stroke
-				(width 0.12)
-				(type solid)
-			)
-			(fill no)
-			(layer "F.SilkS")
-		)
-		(fp_circle
-			(center 0 0)
-			(end 1 0)
-			(stroke
-				(width 0.05)
-				(type solid)
-			)
-			(fill no)
-			(layer "F.CrtYd")
-		)
-		(pad "1" smd circle
-			(at 0 0)
-			(size 1 1)
-			(layers "F.Cu" "F.Mask")
-			(net 6 "+1V2")
-			(pinfunction "1")
-			(pintype "passive")
-		)
-		(embedded_fonts no)
-	)
 	(footprint "PCM_Resistor_SMD_AKL:R_0402_1005Metric"
 		(layer "F.Cu")
@@
 	)
 	(gr_text "1.2V"
-		(at 229.1031 85.400001 0)
+		(at 199.4031 91.900001 0)
 		(layer "F.SilkS")
 		(effects
@@
 	(segment
 		(start 201.6831 93.500001)
+		(end 201.1471 94.036001)
+		(width 0.15)
+		(layer "F.Cu")
+		(net 6)
+	)
+	(segment
+		(start 201.1471 94.036001)
+		(end 199.9391 94.036001)
+		(width 0.15)
+		(layer "F.Cu")
+		(net 6)
+	)
+	(segment
+		(start 201.6831 93.500001)
 		(end 201.7581 93.575001)
 		(width 0.15)
@@
 		(width 0.15)
 		(layer "F.Cu")
+		(net 6)
+	)
+	(segment
+		(start 199.9391 94.036001)
+		(end 198.5031 92.600001)
+		(width 0.15)
+		(layer "F.Cu")
+		(net 6)
+	)
+	(segment
+		(start 198.5031 92.600001)
+		(end 198.5031 91.400001)
+		(width 0.15)
+		(layer "F.Cu")

Commit message: 🔥 Redo the PCB
Parts:
- removed C1, C23: 10uF, Capacitor_SMD:C_0805_2012Metric
- removed C10, C18, C19, C29, C31, C45, C46, C47, C48, C49, C50, C51, C53, C54, C55, C56, C57, C58, C59, C60: 100nF, Capacitor_SMD:C_0402_1005Metric
- removed C11, C14, C17: 100nF/100V, Capacitor_SMD:C_0805_2012Metric
- removed C12, C34, C35, C36, C37, C5, C6: 100nF, Capacitor_SMD:C_0603_1608Metric
- removed C13, C32, C38, C62: 1uF, Capacitor_SMD:C_0603_1608Metric
- removed C15, C16: 10uF/100V, Capacitor_SMD:C_1206_3216Metric
- removed C2: 100nF/50V, Capacitor_SMD:C_0603_1608Metric
- removed C20, C21, C22, C25, C26, C3, C4: 22uF, Capacitor_SMD:C_0805_2012Metric
- removed C24: 4.7nF, Capacitor_SMD:C_0603_1608Metric
- removed C27, C33: 4.7uF, Capacitor_SMD:C_0603_1608Metric
- removed C28: 0.22uF/50V, Capacitor_SMD:C_0805_2012Metric
- removed C39, C40: 12pF, Capacitor_SMD:C_0402_1005Metric
- removed C41, C42, C43, C44: 1uF, Capacitor_SMD:C_0402_1005Metric
- removed C61: 10uF, Capacitor_SMD:C_0603_1608Metric
- removed C7, C8, C9: 1uF/100V, Capacitor_SMD:C_1206_3216Metric
- removed D1: SMF60A, Diode_SMD:D_SOD-123F
- removed D2: PESD2CAN / PESD3V3L2BT, PCM_Package_TO_SOT_SMD_AKL:SOT-23
- removed D3: SRV05-4, PCM_Package_TO_SOT_SMD_AKL:SOT-23-6
- removed DZ1: BZX84-C12, PCM_Package_TO_SOT_SMD_AKL:SOT-23
- removed F2: Fuse, PCM_Fuse_AKL:Fuse_1206_3216Metric
- removed FB1: FerriteBead, Inductor_SMD:L_0805_2012Metric
- removed FL1: ACT32P-102-2P-TL01, PEAK:ACT32P_TDK
- removed J2: Conn_DEBUG_C6, Connector_JST:JST_SHL_SM06B-SHLS-TF_1x06-1MP_P1.00mm_Horizontal
- removed J3: Conn_Buttons, Connector_Molex:Molex_PicoBlade_53261-0471_1x04-1MP_P1.25mm_Horizontal
- removed J4: Conn_DEBUG_P4, Connector_JST:JST_SHL_SM06B-SHLS-TF_1x06-1MP_P1.00mm_Horizontal
- removed J6: Conn_Controller, Connector_Molex:Molex_PicoBlade_53261-0571_1x05-1MP_P1.25mm_Horizontal
- removed L1: 8.2uH, Inductor_SMD:L_Bourns_SRP5030T
- removed L2: 3.9uH, Inductor_SMD:L_APV_ANR4030
- removed L3: 220nH, Inductor_SMD:L_0603_1608Metric
- removed L4: 15uH, Inductor_SMD:L_1210_3225Metric
- removed Q1: DMP10H400SE, PCM_Package_TO_SOT_SMD_AKL:SOT-223-3_TabPin2
- removed Q2: BSS123, PCM_Package_TO_SOT_SMD_AKL:SOT-23
- removed R1: 120R, PCM_Resistor_SMD_AKL:R_0603_1608Metric
- removed R10, R12, R2, R52, R9: 100k, Resistor_SMD:R_0603_1608Metric
- removed R11: 10, Resistor_SMD:R_0805_2012Metric
- removed R13, R44, R45, R51: 10k, PCM_Resistor_SMD_AKL:R_0402_1005Metric
- removed R14, R15, R16, R17, R24, R25: 10k, Resistor_SMD:R_0603_1608Metric
- removed R18: 1M, Resistor_SMD:R_0603_1608Metric
- removed R19: 47k, Resistor_SMD:R_0603_1608Metric
- removed R20, R53, R54, R55, R7: 1k, Resistor_SMD:R_0603_1608Metric
- removed R21, R22, R36, R37, R38, R39, R40, R41, R56: 0, PCM_Resistor_SMD_AKL:R_0402_1005Metric
- removed R23, R48: 4.02k, PCM_Resistor_SMD_AKL:R_0402_1005Metric
- removed R26, R27: 100, Resistor_SMD:R_0603_1608Metric
- removed R28, R29, R8: 0, Resistor_SMD:R_0603_1608Metric
- removed R3: 1k, PCM_Resistor_SMD_AKL:R_0603_1608Metric
- removed R30, R31, R32, R33, R34, R35: 51k, Resistor_SMD:R_0603_1608Metric
- removed R4: 19.1k, Resistor_SMD:R_0603_1608Metric
- removed R42, R43: 4.7k, PCM_Resistor_SMD_AKL:R_0402_1005Metric
- removed R46, R47, R49, R50: 33, PCM_Resistor_SMD_AKL:R_0603_1608Metric
- removed R5, R6: 100k, Resistor_SMD:R_0805_2012Metric
- removed TP1: 5V, TestPoint:TestPoint_Pad_D1.0mm
- removed TP2: 3.3V, TestPoint:TestPoint_Pad_D1.0mm
- removed TP3: 1.2V, TestPoint:TestPoint_Pad_D1.0mm
- removed TP4: LEDA, TestPoint:TestPoint_Pad_D1.0mm
- removed TP6: 3.3VA, TestPoint:TestPoint_Pad_D1.0mm
- removed TP7: VIN, TestPoint:TestPoint_Pad_D1.0mm
- removed TP8: VBUS, TestPoint:TestPoint_Pad_D1.0mm
- removed TP9 (x4): GND, TestPoint:TestPoint_Pad_D1.0mm
- removed U11: LTR-329ALS-01, PEAK:LTR-329ALS-01_LTO
- removed U2: AP63203WU, PCM_Package_TO_SOT_SMD_AKL:TSOT-23-6
- removed U3: MCP2542FDxMF, Package_DFN_QFN:DFN-8-1EP_3x3mm_P0.65mm_EP1.55x2.4mm
- removed U4: TPS62A04ADRL, Package_TO_SOT_SMD:SOT-563
- removed U5: PLMR51635XDDCR, Package_TO_SOT_SMD:SOT-23-6
- removed U6: AP3019AKTR, Package_TO_SOT_SMD:SOT-23-6
- removed U7: W25Q128JVP, Package_SON:WSON-8-1EP_6x5mm_P1.27mm_EP3.4x4.3mm
- removed U8: T117, PCM_Package_DFN_QFN_AKL:DFN-6-1EP_2x2mm_P0.65mm_EP1x1.6mm
- removed U9: 74LVC1G17, PCM_Package_TO_SOT_SMD_AKL:SOT-23-5
- removed X1: ECS-400-10-37B2-CKY-TR, Crystal:Crystal_SMD_2016-4Pin_2.0x1.6mm
Routing:
- net +5V: track 128.8 -> 0.00 mm, vias 10 -> 0
- net +3.3V: track 121.0 -> 0.00 mm, vias 26 -> 0
- net /IO/SDA_MCU: track 77.9 -> 0.00 mm, vias 4 -> 0
- net /IO/SCL_MCU: track 77.6 -> 0.00 mm, vias 4 -> 0
- net Net-(C13-Pad1): track 64.3 -> 0.00 mm, vias 3 -> 0
- net /Connection/Button_D: track 57.1 -> 0.00 mm, vias 3 -> 0
- net /Connection/Button_P: track 54.5 -> 0.00 mm, vias 3 -> 0
- net /Connection/Button_U: track 50.2 -> 0.00 mm, vias 3 -> 0
- net +1V2: track 48.5 -> 0.00 mm, vias 4 -> 0
- net /Connection/TX/CANL: track 38.6 -> 0.00 mm, vias 3 -> 0
- net /MCU/EN: track 37.0 -> 0.00 mm, vias 2 -> 0
- net /Display/LEDA: track 34.5 -> 0.00 mm, vias 2 -> 0
- net /Connection/RX/CANH: track 34.2 -> 0.00 mm, vias 3 -> 0
- net /Display/LED_PWM: track 33.3 -> 0.00 mm, vias 2 -> 0
- net /IO/SW_MCU: track 33.2 -> 0.00 mm, vias 2 -> 0
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- removed copper zone on F.Cu, net +1V2
- removed copper zone on F.Cu, net +3.3V
- removed copper zone on In2.Cu, net +3.3V
- removed copper zone on F.Cu, net +5V
- removed copper zone on In2.Cu, net +5V
- removed copper zone on B.Cu, net GND
- removed copper zone on F.Cu, net GND
- removed copper zone on In1.Cu, net GND
- removed copper zone on In4.Cu, net GND
- removed copper zone on F.Cu, net VBUS
- removed copper zone on In2.Cu, net VBUS
Other:
- board text removed: "1.2V"
- board text removed: "3.3V"
- board text removed: "3.3VA"
- board text removed: "5V"
- board text removed: "Antenna Area"
- board text removed: "BAT+"
- board text removed: "CAN"
- board text removed: "D"
- board text removed: "G"
- board text removed: "GND"
- board text removed: "LED"
- board text removed: "LEDA"
- board text removed: "P"
- board text removed: "R"
- board text removed: "RX"
- board text removed: "S"
- board text removed: "SW"
- board text removed: "T"
- board text removed: "U"
- board text removed: "V"
- board text removed: "VBUS"

Commit message: ✨ Final PCB updates
Parts:
- added C1: 12pF, Capacitor_SMD:C_0402_1005Metric, F.Cu at (204.1, 81.8)
- added C10: 100nF, Capacitor_SMD:C_0402_1005Metric, F.Cu at (216.4, 92.4)
- added C11: 100nF, Capacitor_SMD:C_0402_1005Metric, F.Cu at (210.3, 84.3)
- added C12: 100nF, Capacitor_SMD:C_0402_1005Metric, F.Cu at (208.4, 84.3)
- added C13: 100nF, Capacitor_SMD:C_0402_1005Metric, F.Cu at (201.3, 92.4)
- added C14: 100nF, Capacitor_SMD:C_0402_1005Metric, F.Cu at (216.4, 85.8)
- added C15: 100nF, Capacitor_SMD:C_0402_1005Metric, F.Cu at (209.3, 84.3)
- added C16: 100nF, Capacitor_SMD:C_0402_1005Metric, F.Cu at (216.4, 97.5)
- added C17: 1uF, Capacitor_SMD:C_0402_1005Metric, F.Cu at (216.4, 89.6)
- added C18: 100nF, Capacitor_SMD:C_0402_1005Metric, F.Cu at (216.4, 91.5)
- added C19: 100nF, Capacitor_SMD:C_0402_1005Metric, F.Cu at (216.4, 93.4)
- added C2: 12pF, Capacitor_SMD:C_0402_1005Metric, F.Cu at (208.1, 81.8)
- added C20: 1uF, Capacitor_SMD:C_0402_1005Metric, F.Cu at (216.4, 90.5)
- added C201: 1uF/100V, Capacitor_SMD:C_1206_3216Metric, F.Cu at (192.6, 97.7)
- added C202: 1uF/100V, Capacitor_SMD:C_1206_3216Metric, F.Cu at (190.3, 97.7)
- added C203: 1uF/100V, Capacitor_SMD:C_1206_3216Metric, F.Cu at (188.0, 97.7)
- added C204: 100nF/100V, Capacitor_SMD:C_0805_2012Metric, F.Cu at (187.9, 93.3)
- added C205: 22uF, Capacitor_SMD:C_0805_2012Metric, F.Cu at (194.4, 85.9)
- added C206: 22uF, Capacitor_SMD:C_0805_2012Metric, F.Cu at (194.4, 87.9)
- added C207: 22uF, Capacitor_SMD:C_0805_2012Metric, F.Cu at (194.4, 89.9)
- added C208: 10uF, Capacitor_SMD:C_0805_2012Metric, F.Cu at (189.6, 80.8)
- added C209: 100nF/50V, Capacitor_SMD:C_0603_1608Metric, F.Cu at (189.9, 75.6)
- added C21: 1uF, Capacitor_SMD:C_0402_1005Metric, F.Cu at (216.4, 88.6)
- added C210: 22uF, Capacitor_SMD:C_0805_2012Metric, F.Cu at (193.0, 82.0)
- added C211: 22uF, Capacitor_SMD:C_0805_2012Metric, F.Cu at (195.0, 82.0)
- added C212: 10uF, Capacitor_SMD:C_0805_2012Metric, F.Cu at (227.6, 77.0)
- added C213: 4.7nF, Capacitor_SMD:C_0603_1608Metric, F.Cu at (227.4, 78.8)
- added C214: 22uF, Capacitor_SMD:C_0805_2012Metric, F.Cu at (227.0, 82.8)
- added C215: 22uF, Capacitor_SMD:C_0805_2012Metric, F.Cu at (225.0, 82.8)
- added C216: 1uF, Capacitor_SMD:C_0603_1608Metric, F.Cu at (198.9, 81.5)
- added C217: 4.7uF, Capacitor_SMD:C_0603_1608Metric, F.Cu at (198.9, 83.0)
- added C218: 1uF, Capacitor_SMD:C_0603_1608Metric, F.Cu at (228.5, 87.6)
- added C219: 1uF, Capacitor_SMD:C_0603_1608Metric, F.Cu at (224.3, 87.6)
- added C22: 1uF, Capacitor_SMD:C_0402_1005Metric, F.Cu at (216.4, 87.7)
- added C23: 100nF, Capacitor_SMD:C_0402_1005Metric, F.Cu at (212.6, 98.8)
- added C24: 100nF, Capacitor_SMD:C_0402_1005Metric, F.Cu at (201.3, 88.0)
- added C3: 100nF, Capacitor_SMD:C_0402_1005Metric, F.Cu at (201.3, 93.8)
- added C301: 100nF/100V, Capacitor_SMD:C_0805_2012Metric, F.Cu at (189.6, 129.2)
- added C302: 10uF/100V, Capacitor_SMD:C_1206_3216Metric, F.Cu at (189.2, 124.6)
- added C303: 10uF/100V, Capacitor_SMD:C_1206_3216Metric, F.Cu at (189.2, 122.3)
- added C4: 100nF, Capacitor_SMD:C_0402_1005Metric, F.Cu at (201.3, 86.0)
- added C5: 100nF, Capacitor_SMD:C_0402_1005Metric, F.Cu at (201.3, 85.1)
- added C501: 100nF, Capacitor_SMD:C_0402_1005Metric, F.Cu at (203.0, 98.8)
- added C502: 100nF, Capacitor_SMD:C_0402_1005Metric, F.Cu at (203.9, 98.8)
- added C503: 4.7uF, Capacitor_SMD:C_0603_1608Metric, F.Cu at (228.2, 91.9)
- added C504: 0.22uF/50V, Capacitor_SMD:C_0805_2012Metric, F.Cu at (228.2, 95.1)
- added C6: 100nF, Capacitor_SMD:C_0402_1005Metric, F.Cu at (201.3, 88.9)
- added C601: 100nF, Capacitor_SMD:C_0603_1608Metric, F.Cu at (228.4, 119.8)
- added C602: 100nF, Capacitor_SMD:C_0603_1608Metric, F.Cu at (228.4, 116.8)
- added C603: 100nF, Capacitor_SMD:C_0603_1608Metric, F.Cu at (228.4, 118.3)
- added C604: 100nF, Capacitor_SMD:C_0603_1608Metric, F.Cu at (230.0, 104.1)
- added C605: 100nF, Capacitor_SMD:C_0603_1608Metric, F.Cu at (230.0, 107.1)
- added C606: 100nF, Capacitor_SMD:C_0603_1608Metric, F.Cu at (219.0, 104.6)
- added C607: 100nF/100V, Capacitor_SMD:C_0805_2012Metric, F.Cu at (188.1, 103.9)
- added C608: 1uF, Capacitor_SMD:C_0603_1608Metric, F.Cu at (216.6, 82.1)
- added C609: 100nF, Capacitor_SMD:C_0603_1608Metric, F.Cu at (208.8, 126.1)
- added C610: 1uF, Capacitor_SMD:C_0603_1608Metric, F.Cu at (199.5, 69.8)
- added C7: 100nF, Capacitor_SMD:C_0402_1005Metric, F.Cu at (201.3, 91.4)
- added C701: 1uF, Capacitor_SMD:C_0603_1608Metric, F.Cu at (199.5, 73.8)
- added C702: 10uF, Capacitor_SMD:C_0603_1608Metric, F.Cu at (199.5, 71.3)
- added C8: 100nF, Capacitor_SMD:C_0402_1005Metric, F.Cu at (216.4, 84.8)
- added C9: 100nF, Capacitor_SMD:C_0402_1005Metric, F.Cu at (216.4, 86.7)
- added D301: SMF60A, Diode_SMD:D_SOD-123F, F.Cu at (189.1, 127.0)
- added D302: SRV05-4, PCM_Package_TO_SOT_SMD_AKL:SOT-23-6, F.Cu at (226.9, 127.3)
- added D303: PESD2CAN / PESD3V3L2BT, PCM_Package_TO_SOT_SMD_AKL:SOT-23, F.Cu at (208.8, 119.0)
- added DZ601: BZX84-C12, PCM_Package_TO_SOT_SMD_AKL:SOT-23, F.Cu at (188.9, 107.5)
- added F301: Fuse, PCM_Fuse_AKL:Fuse_1206_3216Metric, F.Cu at (194.1, 129.0)
- added FB201: FerriteBead, Inductor_SMD:L_0805_2012Metric, F.Cu at (201.3, 82.2)
- added J2: Conn_Controller, Connector_Molex:Molex_PicoBlade_53261-0571_1x05-1MP_P1.25mm_Horizontal, F.Cu at (200.1, 124.6)
- added J3: Conn_Buttons, Connector_Molex:Molex_PicoBlade_53261-0471_1x04-1MP_P1.25mm_Horizontal, F.Cu at (217.0, 124.6)
- added J4: Conn_DEBUG_P4, Connector_JST:JST_SHL_SM06B-SHLS-TF_1x06-1MP_P1.00mm_Horizontal, F.Cu at (225.9, 70.6)
- added J5: Conn_DEBUG_C6, Connector_JST:JST_SHL_SM06B-SHLS-TF_1x06-1MP_P1.00mm_Horizontal, F.Cu at (191.8, 70.6)
- added L201: 8.2uH, Inductor_SMD:L_Bourns_SRP5030T, F.Cu at (189.8, 87.8)
- added L202: 3.9uH, Inductor_SMD:L_APV_ANR4030, F.Cu at (193.7, 78.0)
- added L203: 220nH, Inductor_SMD:L_0603_1608Metric, F.Cu at (225.5, 80.3)
- added L501: 15uH, Inductor_SMD:L_1210_3225Metric, F.Cu at (225.2, 91.8)
- added Q601: BSS123, PCM_Package_TO_SOT_SMD_AKL:SOT-23, F.Cu at (192.5, 107.5)
- added Q602: DMP10H400SE, PCM_Package_TO_SOT_SMD_AKL:SOT-223-3_TabPin2, F.Cu at (190.7, 113.7)
- added R1: 0, PCM_Resistor_SMD_AKL:R_0402_1005Metric, F.Cu at (205.5, 84.1)
- added R10: 0, PCM_Resistor_SMD_AKL:R_0402_1005Metric, F.Cu at (211.5, 98.8)
- added R11: 4.02k, PCM_Resistor_SMD_AKL:R_0402_1005Metric, F.Cu at (213.6, 98.8)
- added R12: 10k, PCM_Resistor_SMD_AKL:R_0402_1005Metric, F.Cu at (219.3, 90.1)
- added R13: 10k, PCM_Resistor_SMD_AKL:R_0402_1005Metric, F.Cu at (219.3, 91.1)
- added R14: 10k, PCM_Resistor_SMD_AKL:R_0402_1005Metric, F.Cu at (201.3, 87.0)
- added R15: 4.7k, PCM_Resistor_SMD_AKL:R_0402_1005Metric, F.Cu at (219.3, 92.4)
- added R16: 4.7k, PCM_Resistor_SMD_AKL:R_0402_1005Metric, F.Cu at (219.3, 93.4)
- added R17: 33, PCM_Resistor_SMD_AKL:R_0402_1005Metric, F.Cu at (216.4, 95.6)
- added R18: 33, PCM_Resistor_SMD_AKL:R_0402_1005Metric, F.Cu at (216.4, 96.6)
- added R2: 0, PCM_Resistor_SMD_AKL:R_0402_1005Metric, F.Cu at (206.5, 84.1)
- added R201: 100k, Resistor_SMD:R_0603_1608Metric, F.Cu at (193.8, 91.6)
- added R202: 19.1k, Resistor_SMD:R_0603_1608Metric, F.Cu at (193.0, 93.9)
- added R203: 0, Resistor_SMD:R_0603_1608Metric, F.Cu at (193.2, 126.9)
- added R204: 0, PCM_Resistor_SMD_AKL:R_0402_1005Metric, F.Cu at (224.9, 76.4)
- added R205: 100k, Resistor_SMD:R_0603_1608Metric, F.Cu at (223.0, 80.3)
- added R206: 100k, Resistor_SMD:R_0603_1608Metric, F.Cu at (223.0, 77.3)
- added R207: 0, Resistor_SMD:R_0402_1005Metric, F.Cu at (226.5, 85.9)
- added R3: 10k, PCM_Resistor_SMD_AKL:R_0402_1005Metric, F.Cu at (196.7, 93.7)
- added R301: 100, Resistor_SMD:R_0603_1608Metric, F.Cu at (220.9, 108.1)
- added R302: 100, Resistor_SMD:R_0603_1608Metric, F.Cu at (222.4, 108.1)
- added R303: 0, Resistor_SMD:R_0603_1608Metric, F.Cu at (226.8, 110.0)
- added R304: 0, Resistor_SMD:R_0603_1608Metric, F.Cu at (228.3, 110.0)
- added R305: 1k, Resistor_SMD:R_0603_1608Metric, F.Cu at (225.4, 123.0)
- added R306: 1k, Resistor_SMD:R_0603_1608Metric, F.Cu at (226.9, 123.0)
- added R307: 1k, Resistor_SMD:R_0603_1608Metric, F.Cu at (228.4, 123.0)
- added R308: 100k, Resistor_SMD:R_0603_1608Metric, F.Cu at (229.5, 127.0)
- added R4: 4.02k, PCM_Resistor_SMD_AKL:R_0402_1005Metric, F.Cu at (204.9, 98.8)
- added R5: 0, PCM_Resistor_SMD_AKL:R_0402_1005Metric, F.Cu at (206.1, 98.8)
- added R501: 100k, Resistor_SMD:R_0603_1608Metric, F.Cu at (227.8, 97.6)
- added R502: 10, Resistor_SMD:R_0805_2012Metric, F.Cu at (224.6, 97.8)
- added R6: 0, PCM_Resistor_SMD_AKL:R_0402_1005Metric, F.Cu at (207.1, 98.8)
- added R601: 10k, Resistor_SMD:R_0603_1608Metric, F.Cu at (225.4, 119.8)
- added R602: 10k, Resistor_SMD:R_0603_1608Metric, F.Cu at (225.4, 116.8)
- added R603: 10k, Resistor_SMD:R_0603_1608Metric, F.Cu at (225.4, 118.3)
- added R604: 1k, PCM_Resistor_SMD_AKL:R_0603_1608Metric, F.Cu at (224.9, 104.1)
- added R605: 120R, PCM_Resistor_SMD_AKL:R_0603_1608Metric, F.Cu at (227.5, 103.4)
- added R606: 1k, Resistor_SMD:R_0603_1608Metric, F.Cu at (195.1, 104.2)
- added R607: 10k, Resistor_SMD:R_0603_1608Metric, F.Cu at (193.6, 104.2)
- added R608: 100k, Resistor_SMD:R_0805_2012Metric, F.Cu at (191.9, 103.9)
- added R609: 100k, Resistor_SMD:R_0805_2012Metric, F.Cu at (190.0, 103.9)
- added R610: 1M, Resistor_SMD:R_0603_1608Metric, F.Cu at (208.8, 123.8)
- added R611: 47k, Resistor_SMD:R_0603_1608Metric, F.Cu at (208.8, 122.3)
- added R612: 1k, Resistor_SMD:R_0603_1608Metric, F.Cu at (215.1, 82.1)
- added R7: 0, PCM_Resistor_SMD_AKL:R_0402_1005Metric, F.Cu at (208.1, 98.8)
- added R701: 51k, Resistor_SMD:R_0603_1608Metric, F.Cu at (218.1, 77.3)
- added R702: 51k, Resistor_SMD:R_0603_1608Metric, F.Cu at (218.1, 75.8)
- added R703: 51k, Resistor_SMD:R_0603_1608Metric, F.Cu at (218.1, 74.3)
- added R704: 51k, Resistor_SMD:R_0603_1608Metric, F.Cu at (218.1, 72.8)
- added R705: 51k, Resistor_SMD:R_0603_1608Metric, F.Cu at (218.1, 78.8)
- added R706: 51k, Resistor_SMD:R_0603_1608Metric, F.Cu at (213.6, 82.1)
- added R707: 10k, Resistor_SMD:R_0603_1608Metric, F.Cu at (199.5, 75.3)
- added R708: 10k, Resistor_SMD:R_0603_1608Metric, F.Cu at (212.0, 82.1)
- added R709: 33, PCM_Resistor_SMD_AKL:R_0402_1005Metric, F.Cu at (210.7, 81.6)
- added R710: 33, PCM_Resistor_SMD_AKL:R_0402_1005Metric, F.Cu at (209.7, 81.6)
- added R8: 0, PCM_Resistor_SMD_AKL:R_0402_1005Metric, F.Cu at (209.1, 98.8)
- added R9: 0, PCM_Resistor_SMD_AKL:R_0402_1005Metric, F.Cu at (210.5, 98.8)
- added TP201: 5V, TestPoint:TestPoint_Pad_D1.0mm, F.Cu at (187.4, 83.6)
- added TP202: 3.3V, TestPoint:TestPoint_Pad_D1.0mm, F.Cu at (197.1, 78.1)
- added TP203: 1.2V, TestPoint:TestPoint_Pad_D1.0mm, F.Cu at (223.0, 82.8)
- added TP204: 3.3VA, TestPoint:TestPoint_Pad_D1.0mm, F.Cu at (199.2, 84.9)
- added TP301: VIN, TestPoint:TestPoint_Pad_D1.0mm, F.Cu at (205.4, 128.8)
- added TP302: GND, TestPoint:TestPoint_Pad_D1.0mm, F.Cu at (208.8, 115.9)
- added TP303: VBUS, TestPoint:TestPoint_Pad_D1.0mm, F.Cu at (190.7, 120.2)
- added TP501: LEDA, TestPoint:TestPoint_Pad_D1.0mm, F.Cu at (227.8, 99.4)
- added U2: W25Q128JVP, Package_SON:WSON-8-1EP_6x5mm_P1.27mm_EP3.4x4.3mm, F.Cu at (198.9, 97.0)
- added U201: PLMR51635XDDCR, Package_TO_SOT_SMD:SOT-23-6, F.Cu at (190.6, 93.3)
- added U202: AP63203WU, PCM_Package_TO_SOT_SMD_AKL:TSOT-23-6, F.Cu at (189.1, 78.0)
- added U203: TPS62A04ADRL, Package_TO_SOT_SMD:SOT-563, F.Cu at (224.9, 78.3)
- added U204: LP5910-1.8DRV, PCM_Package_SON_AKL:WSON-6-1EP_2x2mm_P0.65mm_EP1x1.6mm, F.Cu at (226.4, 87.8)
- added U501: AP3019AKTR, Package_TO_SOT_SMD:SOT-23-6, F.Cu at (225.1, 95.1)
- added U601: MCP2542FDxMF, Package_DFN_QFN:DFN-8-1EP_3x3mm_P0.65mm_EP1.55x2.4mm, F.Cu at (227.5, 106.4)
- added U602: 74LVC1G17, PCM_Package_TO_SOT_SMD_AKL:SOT-23-5, F.Cu at (221.5, 104.6)
- added U603: T117, PCM_Package_DFN_QFN_AKL:DFN-6-1EP_2x2mm_P0.65mm_EP1x1.6mm, F.Cu at (208.8, 128.6)
- added U604: LTR-329ALS-01, PEAK:LTR-329ALS-01_LTO, B.Cu at (208.8, 63.9)
- added X1: ECS-400-10-37B2-CKY-TR, Crystal:Crystal_SMD_2016-4Pin_2.0x1.6mm, F.Cu at (206.1, 81.8)
- moved U1 2.00 mm to (208.8, 91.2)
- renumbered U12 to U3
Connections:
- J1 pad 7: +3.3V -> +1V8
- U1 pad 12: /Display/DISPLAY_TE -> unconnected-(U1-GPIO11/ADC-Pad12)
- U1 pad 13: /Display/DISPLAY_RESET -> unconnected-(U1-GPIO12/ADC-Pad13)
- U1 pad 80: unconnected-(U1-GPIO39-Pad80) -> /Display/DISPLAY_TE
- U1 pad 81: unconnected-(U1-GPIO40-Pad81) -> /Display/DISPLAY_RESET
- U1 pad 85: +3.3V -> +1V8
Routing:
- net /IO/SDA_MCU: track 0.00 -> 80.6 mm, vias 0 -> 6
- net /IO/SCL_MCU: track 0.00 -> 79.9 mm, vias 0 -> 6
- net +3.3V: track 0.00 -> 62.7 mm, vias 0 -> 41
- net Net-(C608-Pad1): track 0.00 -> 51.3 mm, vias 0 -> 4
- net /Connection/Button_U: track 0.00 -> 49.3 mm, vias 0 -> 2
- net /Connection/Button_P: track 0.00 -> 49.0 mm, vias 0 -> 2
- net /Connection/Button_D: track 0.00 -> 48.1 mm, vias 0 -> 2
- net +BATT: track 0.00 -> 43.8 mm
- net /MCU/EN: track 0.00 -> 42.2 mm, vias 0 -> 2
- net /Connection/TX/CANL: track 0.00 -> 40.4 mm, vias 0 -> 3
- net +1V8: track 0.00 -> 40.2 mm, vias 0 -> 3
- net /Connection/RX/CANH: track 0.00 -> 38.5 mm, vias 0 -> 3
- net /MCU/RX1: track 0.00 -> 31.5 mm, vias 0 -> 3
- net /MCU/TX1: track 0.00 -> 30.5 mm, vias 0 -> 2
- net /Display/LEDA: track 0.00 -> 29.9 mm, vias 0 -> 2
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- added copper zone on F.Cu, net +1V2
- added copper zone on In2.Cu, net +1V2
- added copper zone on F.Cu, net +1V8
- added copper zone on F.Cu, net +3.3V
- added copper zone on In3.Cu, net +3.3V
- added copper zone on F.Cu, net +5V
- added copper zone on In2.Cu, net +5V
- added copper zone on F.Cu, net /Display/LEDA
- added copper zone on F.Cu, net /Display/LEDK
- added copper zone on B.Cu, net GND
- added copper zone on F.Cu, net GND
- added copper zone on In1.Cu, net GND
- added copper zone on In4.Cu, net GND
- added copper zone on F.Cu, net Net-(U201-SW)
- added copper zone on F.Cu, net Net-(U202-SW)
- added copper zone on F.Cu, net Net-(U501-SW)
- added copper zone on F.Cu, net VBUS
- added copper zone on In2.Cu, net VBUS
Other:
- board text added: "1.2V"
- board text added: "1.8V"
- board text added: "3.3V"
- board text added: "3.3VA"
- board text added: "5V"
- board text added: "BAT"
- board text added: "Buttons"
- board text added: "C6"
- board text added: "CAN"
- board text added: "Controller"
- board text added: "G D P U"
- board text added: "GND"
- board text added: "LED"
- board text added: "P4"
- board text added: "T R G S V"
- board text added: "UART"
- board text added: "VIN"

Commit message: ✨ Final PCB v.1 updates
Parts:
- removed TP203: 1.2V, TestPoint:TestPoint_Pad_D1.0mm
- added R208: 0, PCM_Resistor_SMD_AKL:R_0402_1005Metric, F.Cu at (223.8, 78.5)
- added R209: 0, PCM_Resistor_SMD_AKL:R_0402_1005Metric, F.Cu at (223.8, 77.5)
- L203: value 220nH -> 2.2uH; footprint Inductor_SMD:L_0603_1608Metric -> PCM_Inductor_SMD_AKL:L_1008_2520Metric
- R205, R206: footprint Resistor_SMD:R_0603_1608Metric -> PCM_Resistor_SMD_AKL:R_0402_1005Metric
- U203: value TPS62A04ADRL -> TLV62569DRL
- moved R206 8.66 mm to (229.1, 83.4), turned to 0 degrees
- moved R205 5.25 mm to (227.2, 83.4), turned to 0 degrees
- moved U203 4.46 mm to (229.3, 78.9), turned to -90 degrees
- moved R204 3.32 mm to (223.8, 79.5)
- moved L203 3.06 mm to (228.3, 81.5), turned to 180 degrees
- moved C214 2.50 mm to (224.5, 83.0), turned to 180 degrees
- moved C212 2.33 mm to (226.5, 79.1), turned to 180 degrees
- moved C215 1.84 mm to (224.5, 81.0), turned to 180 degrees
- moved C213 1.54 mm to (226.7, 77.4), turned to 180 degrees
Connections:
- U203 pad 1: GND -> Net-(U203-FB)
- U203 pad 2: Net-(U203-SW) -> GND
- U203 pad 4: Net-(U203-EN) -> Net-(U203-SW)
- U203 pad 5: Net-(U203-FB) -> Net-(U203-EN)
- U203 pad 6: GND -> unconnected-(U203-NC-Pad6)
Routing:
- net /MCU/FB_DCDC: track 0.00 -> 14.3 mm, vias 0 -> 2
- net /MCU/EN_DCDC: track 0.00 -> 13.7 mm, vias 0 -> 2
- net Net-(U203-FB): track 3.76 -> 14.8 mm, vias 0 -> 3
- net Net-(U203-EN): track 1.20 -> 9.27 mm, vias 0 -> 2
- net +3.3V: track 62.7 -> 58.7 mm, vias 41 -> 43
- net Net-(U203-SW): track 1.33 -> 0.00 mm
- net GND: vias 63 -> 103
- added copper zone on F.Cu, net Net-(U203-SW)
